File: kicad/schematics/31_motor_kern.kicad_sch (KiCad schematic)
At the start: 2 parts, among them Q1 CircuitBreaker_2P

Commit message: Schema's
00 toplevel stabiel
10 wisselstroom met subbladen stabiel
15 energieconversie stabiel
31 motor kern stabiel
32 motor sensoren stabiel
50 sensoren stabiel
Parts:
- removed A2: Galvanische Isolator, symbol falkor-electrical:galvanic_isolator
- removed Q1: CircuitBreaker_2P, symbol falkor-electrical:CircuitBreaker_2P
- added G1: Dynamo, symbol falkor-electrical:dynamo
- added K1: Relay_SPST-NO, symbol falkor-electrical:Relay_SPST-NO
- added M1: Startmotor, symbol falkor-electrical:startmotor
Connections:
- new net: K1.14, M1.1 (DC+)
- new net DC_NEG_ALT: G1.2 (D-)
- new net DC_NEG_START: K1.A1, M1.2 (DC-)
- new net DC_POS_ALT: G1.1 (B+)
- new net DC_POS_START: K1.13
- new net SIG_ALT_ACTIVE: G1.3 (D+)
- new net SIG_ALT_RPM: G1.4 (W)
- new net SIG_ENG_START: K1.A2
- no-connect marks 0 -> 2
Other:
- note added: "Controleren of huidige dynamo Falkor deze aansluiting heeft"
- note added: "Mechanisch verbonden via motorblok naar ENG_CASE (zie 90 referenties)"
- note added: "Niet aangesloten, DC-DC lader signaleert zelf of dynamo laadstroom afgeeft"
