File: kicad/schematics/90_referentiepunten.kicad_sch (KiCad schematic)
At the start: 0 parts

Commit message: Schema's
00 toplevel stabiel
10 wisselstroom met subbladen stabiel
15 energieconversie stabiel
31 motor kern stabiel
32 motor sensoren stabiel
50 sensoren stabiel
Changed lines of the file:
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@@
-	)
-	(no_connect
-		(at 52.07 83.82)
 	)
 	(no_connect
@@
 	)
 	(no_connect
+		(at 45.72 96.52)
+	)
+	(no_connect
 		(at 52.07 63.5)
 	)
@@
 		(shape passive)
 		(at 53.34 52.07 180)
-		(effects
-			(font
-				(size 1.27 1.27)
-			)
-			(justify right)
-		)
-	)
-	(hierarchical_label "DC_NEG_CHARGE"
-		(shape passive)
-		(at 52.07 83.82 180)
 		(effects
 			(font
@@
 		)
 	)
+	(hierarchical_label "PE"
+		(shape passive)
+		(at 45.72 96.52 0)
+		(effects
+			(font
+				(size 1.27 1.27)
+			)
+			(justify left)
+		)
+	)

Commit message: 90_referentiepunten stabiel
Parts:
- added Z1: Motorblok, symbol falkor-electrical:engine_case
Connections:
- net DC_NEG_ALTN: now also Z1.3 (GND)
- net DC_NEG_HOUSE: now also Z1.1 (GND)
- net DC_NEG_START: now also Z1.2 (GND)
- net PE: now also Z1.4 (GND)
- no-connect marks 4 -> 0
Changed lines of the file:
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@@
 		(company "Gerard van Konijnenburg")
 	)
-	(no_connect
-		(at 53.34 52.07)
+	(wire
+		(pts
+			(xy 63.5 63.5) (xy 73.66 63.5)
+		)
+		(stroke
+			(width 0)
+			(type default)
+		)
 	)
-	(no_connect
-		(at 52.07 73.66)
+	(wire
+		(pts
+			(xy 63.5 68.58) (xy 73.66 68.58)
+		)
+		(stroke
+			(width 0)
+			(type default)
+		)
 	)
-	(no_connect
-		(at 45.72 96.52)
+	(wire
+		(pts
+			(xy 63.5 53.34) (xy 73.66 53.34)
+		)
+		(stroke
+			(width 0)
+			(type default)
+		)
 	)
-	(no_connect
-		(at 52.07 63.5)
+	(wire
+		(pts
+			(xy 63.5 58.42) (xy 73.66 58.42)
+		)
+		(stroke
+			(width 0)
+			(type default)
+		)
 	)
 	(hierarchical_label "DC_NEG_HOUSE"
 		(shape passive)
-		(at 53.34 52.07 180)
+		(at 63.5 53.34 180)
 		(effects
 			(font
@@
 	(hierarchical_label "DC_NEG_START"
 		(shape passive)
-		(at 52.07 63.5 180)
+		(at 63.5 58.42 180)
 		(effects
 			(font
@@
 	(hierarchical_label "PE"
 		(shape passive)
-		(at 45.72 96.52 0)
-		(effects
-			(font
-				(size 1.27 1.27)
-			)
-			(justify left)
-		)
-	)
-	(hierarchical_label "DC_NEG_ALTN"
-		(shape passive)
-		(at 52.07 73.66 180)
+		(at 63.5 68.58 180)
 		(effects
 			(font
@@
 		)
 	)
+	(hierarchical_label "DC_NEG_ALTN"
+		(shape passive)
+		(at 63.5 63.5 180)
+		(effects
+			(font
+				(size 1.27 1.27)
+			)
+			(justify right)
+		)
+	)
+	(symbol
+		(lib_id "falkor-electrical:engine_case")
+		(at 82.55 60.96 0)
+		(unit 1)
+		(body_style 1)
+		(exclude_from_sim no)
+		(in_bom yes)
+		(on_board yes)
+		(in_pos_files yes)
+		(dnp no)
+		(fields_autoplaced yes)
+		(property "Reference" "Z1"
+			(at 90.17 59.6899 0)
+			(hide yes)
+			(show_name no)
+			(do_not_autoplace no)
+			(effects
+				(font
+					(size 1.27 1.27)
+				)
+				(justify left)
+			)
+		)
+		(property "Value" "Motorblok"
+			(at 90.17 62.2299 0)
+			(show_name no)
+			(do_not_autoplace no)
+			(effects
+				(font
+					(size 1.27 1.27)
+				)
+				(justify left)
+			)
+		)
+		(property "Footprint" ""
+			(at 82.55 60.96 0)
+			(hide yes)
+			(show_name no)
+			(do_not_autoplace no)
+			(effects
+				(font
+					(size 1.27 1.27)
+				)
+			)
+		)
+		(property "Datasheet" ""
+			(at 82.55 60.96 0)
+			(hide yes)
+			(show_name no)
+			(do_not_autoplace no)
+			(effects
+				(font
+					(size 1.27 1.27)
+				)
+			)
+		)
+		(property "Description" ""
+			(at 82.55 60.96 0)
+			(hide yes)
+			(show_name no)
+			(do_not_autoplace no)
+			(effects
+				(font
+					(size 1.27 1.27)
+				)
+			)
+		)
+		(pin "4"
+		)
+		(pin "1"
+		)
+		(pin "3"
+		)
+		(pin "2"
+		)
+		(instances
+			(project "falkor-electrical"
+				(path "/9f36350e-4cf0-4a74-b7c3-6abcdf4429c7/516a7b53-bc29-4762-af31-31effd98f175"
+					(reference "Z1")
+					(unit 1)
+				)
+			)
+		)
+	)
