File: kicad/schematics/90_referentiepunten.kicad_sch (KiCad schematic)
At the start: 1 part

Commit message: Vervolg 21_laden_opslag_distributie
Connections:
- net DC_NEG_HOUSE renamed GND
Changed lines of the file:
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@@
 		)
 	)
-	(hierarchical_label "DC_NEG_HOUSE"
+	(hierarchical_label "GND"
 		(shape passive)
 		(at 63.5 53.34 180)
