File: kicad/schematics/30_motor.kicad_sch (KiCad schematic)
At the start: 6 parts

Commit message: Schema's
00 toplevel stabiel
10 wisselstroom met subbladen stabiel
15 energieconversie stabiel
31 motor kern stabiel
32 motor sensoren stabiel
50 sensoren stabiel
Parts:
- removed T22, T23: (no value), symbol falkor-electrical:IF_Passief
- removed T24, T25, T26, T27: (no value), symbol falkor-electrical:IF_Power_Input
Other:
- added sheet 31 Motor kern (31_motor_kern.kicad_sch)
- added sheet 32 Motor sensoren (32_motor_sensoren.kicad_sch)

Commit message: eerste opzet 21_laden_opslag_distributie
Changed lines of the file:
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@@
 	(sheet
 		(at 88.9 63.5)
-		(size 38.1 25.4)
+		(size 38.1 12.7)
 		(exclude_from_sim no)
 		(in_bom yes)
@@
 		)
 		(property "Sheetname" "32 Motor sensoren"
-			(at 88.9 62.7884 0)
+			(at 88.9 62.7376 0)
 			(show_name no)
 			(do_not_autoplace no)
@@
 		)
 		(property "Sheetfile" "32_motor_sensoren.kicad_sch"
-			(at 88.9 89.4846 0)
+			(at 88.9 76.8354 0)
 			(hide yes)
 			(show_name no)
@@
 	(sheet
 		(at 88.9 25.4)
-		(size 38.1 25.4)
+		(size 38.1 12.7)
 		(exclude_from_sim no)
 		(in_bom yes)
@@
 		)
 		(property "Sheetname" "31 Motor kern"
-			(at 88.9 24.6884 0)
+			(at 88.9 24.6376 0)
 			(show_name no)
 			(do_not_autoplace no)
@@
 		)
 		(property "Sheetfile" "31_motor_kern.kicad_sch"
-			(at 88.9 51.3846 0)
+			(at 88.9 38.7354 0)
 			(hide yes)
 			(show_name no)
