File: kicad/schematics/32_motor_sensoren.kicad_sch (KiCad schematic)
At the start: 4 parts

Commit message: eerste opzet 21_laden_opslag_distributie
Parts:
- S13: renamed from S14; value Sensor -> Oliedruk
- S14: renamed from S15; value Sensor -> Olietemperatuur
- S15: renamed from S16; value Sensor -> RPM
- S16: renamed from S17; value Sensor -> Watertemperatuur
Changed lines of the file:
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@@
 		(dnp no)
 		(fields_autoplaced yes)
-		(property "Reference" "S15"
+		(property "Reference" "S14"
 			(at 57.175 58.42 0)
 			(show_name no)
@@
 			)
 		)
-		(property "Value" "Sensor"
+		(property "Value" "Olietemperatuur"
 			(at 57.175 60.96 0)
 			(show_name no)
@@
 			(project "falkor-electrical"
 				(path "/9f36350e-4cf0-4a74-b7c3-6abcdf4429c7/13c187e7-31a7-4196-98a6-1bea17f9214f/113436b5-6a1f-4212-9384-dca55b119f49"
-					(reference "S15")
+					(reference "S14")
 					(unit 1)
 				)
@@
 		(dnp no)
 		(fields_autoplaced yes)
-		(property "Reference" "S17"
+		(property "Reference" "S16"
 			(at 57.175 96.52 0)
 			(show_name no)
@@
 			)
 		)
-		(property "Value" "Sensor"
+		(property "Value" "Watertemperatuur"
 			(at 57.175 99.06 0)
 			(show_name no)
@@
 			(project "falkor-electrical"
 				(path "/9f36350e-4cf0-4a74-b7c3-6abcdf4429c7/13c187e7-31a7-4196-98a6-1bea17f9214f/113436b5-6a1f-4212-9384-dca55b119f49"
-					(reference "S17")
+					(reference "S16")
 					(unit 1)
 				)
@@
 		(dnp no)
 		(fields_autoplaced yes)
-		(property "Reference" "S16"
+		(property "Reference" "S15"
 			(at 57.175 76.2 0)
 			(show_name no)
@@
 			)
 		)
-		(property "Value" "Sensor"
+		(property "Value" "RPM"
 			(at 57.175 78.74 0)
 			(show_name no)
@@
 			(project "falkor-electrical"
 				(path "/9f36350e-4cf0-4a74-b7c3-6abcdf4429c7/13c187e7-31a7-4196-98a6-1bea17f9214f/113436b5-6a1f-4212-9384-dca55b119f49"
-					(reference "S16")
+					(reference "S15")
 					(unit 1)
 				)
@@
 		(dnp no)
 		(fields_autoplaced yes)
-		(property "Reference" "S14"
+		(property "Reference" "S13"
 			(at 57.175 38.1 0)
 			(show_name no)
@@
 			)
 		)
-		(property "Value" "Sensor"
+		(property "Value" "Oliedruk"
 			(at 57.175 40.64 0)
 			(show_name no)
@@
 			(project "falkor-electrical"
 				(path "/9f36350e-4cf0-4a74-b7c3-6abcdf4429c7/13c187e7-31a7-4196-98a6-1bea17f9214f/113436b5-6a1f-4212-9384-dca55b119f49"
-					(reference "S14")
-					(unit 1)
-				)
+					(reference "S13")
+					(unit 1)
+				)
