File: kicad/schematics/12_ac_verbruikers.kicad_sch (KiCad schematic)
At the start: 6 parts

Commit message: Vervolg 21_laden_opslag_distributie
Parts:
- renumbered T14 to T10, T9 to T5, T10 to T6, T11 to T7, T12 to T8, T13 to T9
Changed lines of the file:
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@@
 		(dnp no)
 		(fields_autoplaced yes)
-		(property "Reference" "T13"
+		(property "Reference" "T9"
 			(at 106.68 87.6299 90)
 			(show_name no)
@@
 			(project "falkor-electrical"
 				(path "/9f36350e-4cf0-4a74-b7c3-6abcdf4429c7/af7fc4f0-c6f0-4760-b6f1-dc4abcc6f651/69803f14-c382-48bb-abea-83bd565ceb0c"
-					(reference "T13")
+					(reference "T9")
 					(unit 1)
 				)
@@
 		(dnp no)
 		(fields_autoplaced yes)
-		(property "Reference" "T10"
+		(property "Reference" "T6"
 			(at 106.68 66.0399 90)
 			(show_name no)
@@
 			(project "falkor-electrical"
 				(path "/9f36350e-4cf0-4a74-b7c3-6abcdf4429c7/af7fc4f0-c6f0-4760-b6f1-dc4abcc6f651/69803f14-c382-48bb-abea-83bd565ceb0c"
-					(reference "T10")
+					(reference "T6")
 					(unit 1)
 				)
@@
 		(dnp no)
 		(fields_autoplaced yes)
-		(property "Reference" "T14"
+		(property "Reference" "T10"
 			(at 106.68 91.4399 90)
 			(show_name no)
@@
 			(project "falkor-electrical"
 				(path "/9f36350e-4cf0-4a74-b7c3-6abcdf4429c7/af7fc4f0-c6f0-4760-b6f1-dc4abcc6f651/69803f14-c382-48bb-abea-83bd565ceb0c"
-					(reference "T14")
+					(reference "T10")
 					(unit 1)
 				)
@@
 		(dnp no)
 		(fields_autoplaced yes)
-		(property "Reference" "T9"
+		(property "Reference" "T5"
 			(at 106.68 63.4999 90)
 			(show_name no)
@@
 			(project "falkor-electrical"
 				(path "/9f36350e-4cf0-4a74-b7c3-6abcdf4429c7/af7fc4f0-c6f0-4760-b6f1-dc4abcc6f651/69803f14-c382-48bb-abea-83bd565ceb0c"
-					(reference "T9")
+					(reference "T5")
 					(unit 1)
 				)
@@
 		(dnp no)
 		(fields_autoplaced yes)
-		(property "Reference" "T12"
+		(property "Reference" "T8"
 			(at 106.68 85.0899 90)
 			(show_name no)
@@
 			(project "falkor-electrical"
 				(path "/9f36350e-4cf0-4a74-b7c3-6abcdf4429c7/af7fc4f0-c6f0-4760-b6f1-dc4abcc6f651/69803f14-c382-48bb-abea-83bd565ceb0c"
-					(reference "T12")
+					(reference "T8")
 					(unit 1)
 				)
@@
 		(dnp no)
 		(fields_autoplaced yes)
-		(property "Reference" "T11"
+		(property "Reference" "T7"
 			(at 106.68 69.8499 90)
 			(show_name no)
@@
 			(project "falkor-electrical"
 				(path "/9f36350e-4cf0-4a74-b7c3-6abcdf4429c7/af7fc4f0-c6f0-4760-b6f1-dc4abcc6f651/69803f14-c382-48bb-abea-83bd565ceb0c"
-					(reference "T11")
-					(unit 1)
-				)
+					(reference "T7")
+					(unit 1)
+				)
