File: kicad/schematics/15_energieconversie.kicad_sch (KiCad schematic)
At the start: 1 part

Commit message: Vervolg 21_laden_opslag_distributie
Connections:
- net DC_NEG_HOUSE renamed DC_NEG_PWR_CONV
- net DC_POS_HOUSE renamed DC_POS_PWR_CONV
Changed lines of the file:
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@@
 		)
 	)
-	(hierarchical_label "DC_POS_HOUSE"
+	(hierarchical_label "DC_POS_PWR_CONV"
 		(shape bidirectional)
 		(at 161.29 25.4 0)
@@
 		)
 	)
-	(hierarchical_label "DC_NEG_HOUSE"
+	(hierarchical_label "DC_NEG_PWR_CONV"
 		(shape bidirectional)
 		(at 161.29 27.94 0)
