File: kicad/falkor-electrical.kicad_sch (KiCad schematic)
At the start: 2 parts, among them J1 Conn_01x03_Pin

Commit message: Vervolg 21_laden_opslag_distributie
Other:
- sheet 15 Energieconversie ports: added DC_NEG_PWR_CONV, DC_POS_PWR_CONV; removed DC_NEG_HOUSE, DC_POS_HOUSE
- sheet 20 Gelijkstroom ports: added DC_NEG_PWR_CONV, DC_POS_PWR_CONV, GND; removed DC_NEG_HOUSE, DC_POS_HOUSE
- sheet 90 Referentiepunten ports: added GND; removed DC_NEG_HOUSE
Changed lines of the file:
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@@
 	)
 	(junction
-		(at 185.42 55.88)
-		(diameter 0)
-		(color 0 0 0 0)
-	)
-	(junction
-		(at 177.8 73.66)
+		(at 177.8 71.12)
 		(diameter 0)
 		(color 0 0 0 0)
@@
 	(wire
 		(pts
-			(xy 185.42 55.88) (xy 190.5 55.88)
+			(xy 165.1 55.88) (xy 190.5 55.88)
 		)
 		(stroke
@@
 	(wire
 		(pts
-			(xy 177.8 73.66) (xy 190.5 73.66)
+			(xy 177.8 71.12) (xy 190.5 71.12)
 		)
 		(stroke
@@
 	(wire
 		(pts
+			(xy 185.42 76.2) (xy 185.42 88.9)
+		)
+		(stroke
+			(width 0)
+			(type default)
+		)
+	)
+	(wire
+		(pts
 			(xy 228.6 132.08) (xy 241.3 132.08)
 		)
@@
 	(wire
 		(pts
-			(xy 165.1 73.66) (xy 177.8 73.66)
+			(xy 187.96 73.66) (xy 185.42 76.2)
+		)
+		(stroke
+			(width 0)
+			(type default)
+		)
+	)
+	(wire
+		(pts
+			(xy 165.1 71.12) (xy 177.8 71.12)
 		)
 		(stroke
@@
 	(wire
 		(pts
-			(xy 165.1 55.88) (xy 185.42 55.88)
-		)
-		(stroke
-			(width 0)
-			(type default)
-		)
-	)
-	(wire
-		(pts
 			(xy 123.19 66.04) (xy 127 66.04)
 		)
@@
 	(wire
 		(pts
+			(xy 177.8 71.12) (xy 177.8 114.3)
+		)
+		(stroke
+			(width 0)
+			(type default)
+		)
+	)
+	(wire
+		(pts
 			(xy 231.14 53.34) (xy 233.68 50.8)
 		)
@@
 	(wire
 		(pts
-			(xy 185.42 55.88) (xy 185.42 88.9)
+			(xy 187.96 73.66) (xy 190.5 73.66)
 		)
 		(stroke
@@
 		(pts
 			(xy 246.38 73.66) (xy 247.65 74.93)
-		)
-		(stroke
-			(width 0)
-			(type default)
-		)
-	)
-	(wire
-		(pts
-			(xy 177.8 73.66) (xy 177.8 114.3)
 		)
 		(stroke
@@
 			)
 		)
-		(pin "DC_NEG_HOUSE" passive
+		(pin "GND" passive
 			(at 190.5 91.44 180)
 			(effects
@@
 			)
 		)
-		(pin "DC_NEG_HOUSE" bidirectional
+		(pin "DC_NEG_PWR_CONV" bidirectional
 			(at 165.1 55.88 0)
 			(effects
@@
 			)
 		)
-		(pin "DC_POS_HOUSE" bidirectional
+		(pin "DC_POS_PWR_CONV" bidirectional
 			(at 165.1 53.34 0)
 			(effects
@@
 		)
 		(pin "N2K" passive
-			(at 165.1 73.66 0)
+			(at 165.1 71.12 0)
 			(effects
 				(font
@@
 			)
 		)
-		(pin "DC_NEG_HOUSE" bidirectional
+		(pin "DC_NEG_PWR_CONV" bidirectional
 			(at 190.5 55.88 180)
 			(effects
@@
 		)
 		(pin "N2K" passive
-			(at 190.5 73.66 180)
+			(at 190.5 71.12 180)
 			(effects
 				(font
@@
 			)
 		)
-		(pin "DC_POS_HOUSE" bidirectional
+		(pin "DC_POS_PWR_CONV" bidirectional
 			(at 190.5 53.34 180)
 			(effects
 				(font
+					(size 1.27 1.27)
+				)
+				(justify left)
+			)
+		)
+		(pin "GND" output
+			(at 190.5 73.66 180)
+			(effects
+				(font
